File: pcb/so-dimm-esp32-cm.kicad_pcb (KiCad board)
At the start: 4 copper layers, 67.6 x 31.1 mm, 37 parts, among them IC1 PI4IOE5V9535LEX, IC2 PI4IOE5V9535LEX, J1 SODIMM-200, U2 ESP32-S2-SOLO

Commit message: Ignored thermal-relief + changed ESP32-S2 to be ESP32-S3-N8
Parts:
- U2: value ESP32-S2-SOLO -> ESP32-S3-WROOM-1-N8
Changed lines of the file:
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@@
         (effects (font (size 1 1) (thickness 0.15)))
     )
-    (fp_text value "ESP32-S2-SOLO" (at 0 12 90) (layer "F.Fab")
+    (fp_text value "ESP32-S3-WROOM-1-N8" (at 0 12 90) (layer "F.Fab")
         (effects (font (size 1 1) (thickness 0.15)))
     )

Commit message: Added assembly file + bom XLSX File (K&G)
Other:
- board text added: "Use for Panelizing"
Changed lines of the file:
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@@
         (effects (font (size 0.6 0.6) (thickness 0.15)))
     )
-    (fp_text value "1uF" (at 0 1.43) (layer "F.Fab")
+    (fp_text value "1uF" (at 3.048 0) (layer "F.Fab")
         (effects (font (size 1 1) (thickness 0.15)))
     )
@@
         (effects (font (size 0.6 0.6) (thickness 0.15)))
     )
-    (fp_text value "10k" (at 0 1.43) (layer "F.Fab")
+    (fp_text value "10k" (at 0 -1.27) (layer "F.Fab")
         (effects (font (size 1 1) (thickness 0.15)))
     )
@@
         (effects (font (size 0.6 0.6) (thickness 0.15)))
     )
-    (fp_text value "LED_RED" (at 0 1.43 90) (layer "F.Fab")
+    (fp_text value "LED_RED" (at -2.41905 -0.7366 180) (layer "F.Fab")
         (effects (font (size 1 1) (thickness 0.15)))
     )
@@
         (effects (font (size 0.6 0.6) (thickness 0.15)))
     )
-    (fp_text value "10k" (at 0 1.43 90) (layer "F.Fab")
+    (fp_text value "10k" (at 3.175 -0.127 90) (layer "F.Fab")
         (effects (font (size 1 1) (thickness 0.15)))
     )
@@
         (effects (font (size 0.6 0.6) (thickness 0.15)))
     )
-    (fp_text value "10k" (at 0 1.43 90) (layer "F.Fab")
+    (fp_text value "10k" (at 3.175 0 90) (layer "F.Fab")
         (effects (font (size 1 1) (thickness 0.15)))
     )
@@
         (effects (font (size 0.6 0.6) (thickness 0.15)))
     )
-    (fp_text value "1k" (at 0 1.43 90) (layer "F.Fab")
+    (fp_text value "1k" (at 0 -1.6256 180) (layer "F.Fab")
         (effects (font (size 1 1) (thickness 0.15)))
     )
@@
         (effects (font (size 0.6 0.6) (thickness 0.15)))
     )
-    (fp_text value "DNP" (at 0 1.43) (layer "F.Fab")
+    (fp_text value "DNP" (at 0 1.43) (layer "F.Fab") hide
         (effects (font (size 1 1) (thickness 0.15)))
     )
@@
         (effects (font (size 1.27 1.27) (thickness 0.254)))
     )
+    (fp_text user "${REFERENCE}" (at 0 0 unlocked) (layer "F.Fab")
+        (effects (font (size 1 1) (thickness 0.15)))
+    )
     (fp_line (start -3.675 -4.15) (end -2.2 -4.15)
       (stroke (width 0.2) (type solid)) (layer "F.SilkS"))
@@
         (effects (font (size 0.6 0.6) (thickness 0.15)))
     )
-    (fp_text value "10k/DNP" (at 0 1.43) (layer "F.Fab")
+    (fp_text value "10k/DNP" (at 0 1.43) (layer "F.Fab") hide
         (effects (font (size 1 1) (thickness 0.15)))
     )
@@
         (effects (font (size 0.6 0.6) (thickness 0.15)))
     )
-    (fp_text value "10k" (at 0 1.43 90) (layer "F.Fab")
+    (fp_text value "10k" (at -2.794 0 90) (layer "F.Fab")
         (effects (font (size 1 1) (thickness 0.15)))
     )
@@
     )
     (fp_text user "${REFERENCE}" (at 0 0) (layer "F.Fab")
-        (effects (font (size 1.27 1.27) (thickness 0.254)))
+        (effects (font (size 1 1) (thickness 0.15)))
     )
     (fp_line (start -3.675 -4.15) (end -2.2 -4.15)
@@
         (effects (font (size 0.6 0.6) (thickness 0.15)))
     )
-    (fp_text value "10k" (at 0 1.43) (layer "F.Fab")
+    (fp_text value "10k" (at 0.127 -1.397) (layer "F.Fab")
         (effects (font (size 1 1) (thickness 0.15)))
     )
@@
         (effects (font (size 0.6 0.6) (thickness 0.15)))
     )
-    (fp_text value "0.1uF" (at 0 1.43) (layer "F.Fab")
+    (fp_text value "0.1uF" (at 3.683 0) (layer "F.Fab")
         (effects (font (size 1 1) (thickness 0.15)))
     )
@@
         (effects (font (size 0.6 0.6) (thickness 0.15)))
     )
-    (fp_text value "10k" (at 0 1.43 90) (layer "F.Fab")
+    (fp_text value "10k" (at -2.794 0 90) (layer "F.Fab")
         (effects (font (size 1 1) (thickness 0.15)))
     )
@@
         (effects (font (size 0.6 0.6) (thickness 0.15)))
     )
-    (fp_text value "0.1uF/DNP" (at 0 3.556) (layer "F.Fab")
+    (fp_text value "0.1uF/DNP" (at 0 3.556) (layer "F.Fab") hide
         (effects (font (size 1 1) (thickness 0.15)))
     )
@@
         (effects (font (size 0.6 0.6) (thickness 0.15)))
     )
-    (fp_text value "0.1uF" (at 0 1.43 90) (layer "F.Fab")
+    (fp_text value "0.1uF" (at 3.683 0 90) (layer "F.Fab")
         (effects (font (size 1 1) (thickness 0.15)))
     )
@@
         (effects (font (size 1 1) (thickness 0.15)))
     )
-    (fp_text value "MountingHole_Pad" (at 0 3.7) (layer "F.Fab")
+    (fp_text value "MountingHole_Pad" (at 0 3.7) (layer "F.Fab") hide
         (effects (font (size 1 1) (thickness 0.15)))
     )
-    (fp_text user "${REFERENCE}" (at 0 0) (layer "F.Fab")
+    (fp_text user "${REFERENCE}" (at 0 0) (layer "F.Fab") hide
         (effects (font (size 1 1) (thickness 0.15)))
     )
@@
         (effects (font (size 0.6 0.6) (thickness 0.15)))
     )
-    (fp_text value "10uF" (at 0 1.43) (layer "F.Fab")
+    (fp_text value "10uF" (at 3.683 0) (layer "F.Fab")
         (effects (font (size 1 1) (thickness 0.15)))
     )
@@
         (effects (font (size 0.6 0.6) (thickness 0.15)))
     )
-    (fp_text value "10k" (at 0 1.43) (layer "F.Fab")
+    (fp_text value "10k" (at 3.048 0) (layer "F.Fab")
         (effects (font (size 1 1) (thickness 0.15)))
     )
@@
         (effects (font (size 0.6 0.6) (thickness 0.15)))
     )
-    (fp_text value "0.1uF" (at 0 1.43 90) (layer "F.Fab")
+    (fp_text value "0.1uF" (at 3.683 -0.127 90) (layer "F.Fab")
         (effects (font (size 1 1) (thickness 0.15)))
     )
@@
         (effects (font (size 1 1) (thickness 0.15)))
     )
-    (fp_text value "ESP32-S3-WROOM-1-N8" (at 0 12 90) (layer "F.Fab")
+    (fp_text value "ESP32-S3-WROOM-1-N8" (at 1.384 -1.402 180) (layer "F.Fab")
         (effects (font (size 1 1) (thickness 0.15)))
     )
@@
         (effects (font (size 1 1) (thickness 0.15)))
     )
-    (fp_text user "${REFERENCE}" (at 0 0 90) (layer "F.Fab")
+    (fp_text user "${REFERENCE}" (at 2.654 0.884 180) (layer "F.Fab")
         (effects (font (size 1 1) (thickness 0.15)))
     )
@@
   (gr_arc (start 183.025346 90.077001) (mid 181.025346 88.077001) (end 183.025346 86.077001)
     (stroke (width 0.15) (type solid)) (layer "Edge.Cuts"))
+  (gr_line (start 116.332 96.52) (end 116.967 96.139)
+    (stroke (width 0.1) (type default)) (layer "F.Fab"))
+  (gr_line (start 116.332 95.758) (end 116.967 96.139)
+    (stroke (width 0.1) (type default)) (layer "F.Fab"))
+  (gr_line (start 114.554 96.139) (end 116.967 96.139)
+    (stroke (width 0.1) (type default)) (layer "F.Fab"))
   (gr_text "199" (at 182.245 107.569 90) (layer "F.Cu")
     (effects (font (size 0.6 0.6) (thickness 0.15)) (justify left bottom))
@@
     (effects (font (size 0.6 0.6) (thickness 0.15)))
   )
-  (dimension (type aligned) (layer "F.SilkS")
+  (gr_text "Use for Panelizing" (at 100.076 96.52) (layer "F.Fab")
+    (effects (font (size 1 1) (thickness 0.15)) (justify left bottom))
+  )
+  (dimension (type aligned) (layer "F.Fab")
     (pts (xy 115.473 108.077001) (xy 131.175346 108.077001))
     (height 5.460999)
-    (gr_text "15.7023 mm" (at 123.324173 112.388) (layer "F.SilkS")
+    (gr_text "15.7023 mm" (at 123.324173 112.388) (layer "F.Fab")
       (effects (font (size 1 1) (thickness 0.15)))
     )
@@
     (style (thickness 0.15) (arrow_length 1.27) (text_position_mode 0) (extension_height 0.58642) (extension_offset 0.5) keep_text_aligned)
   )
-  (dimension (type aligned) (layer "F.SilkS")
+  (dimension (type aligned) (layer "F.Fab")
     (pts (xy 132.175346 108.077001) (xy 183.007 108.077))
     (height 5.467206)
-    (gr_text "50.8317 mm" (at 157.591173 112.394206 2.254334674e-06) (layer "F.SilkS")
+    (gr_text "50.8317 mm" (at 157.591173 112.394206 2.254334674e-06) (layer "F.Fab")
       (effects (font (size 1 1) (thickness 0.15)))
     )
@@
     (style (thickness 0.15) (arrow_length 1.27) (text_position_mode 0) (extension_height 0.58642) (extension_offset 0.5) keep_text_aligned)
   )
-  (dimension (type aligned) (layer "F.SilkS")
+  (dimension (type aligned) (layer "F.Fab")
     (pts (xy 183.025345 77.677001) (xy 115.425346 77.677001))
     (height 5.160001)
-    (gr_text "67.6000 mm" (at 149.225345 71.367) (layer "F.SilkS")
+    (gr_text "67.6000 mm" (at 149.225345 71.367) (layer "F.Fab")
       (effects (font (size 1 1) (thickness 0.15)))
     )
@@
     (style (thickness 0.15) (arrow_length 1.27) (text_position_mode 0) (extension_height 0.58642) (extension_offset 0.5) keep_text_aligned)
   )
-  (dimension (type aligned) (layer "F.SilkS")
+  (dimension (type aligned) (layer "F.Fab")
     (pts (xy 182.275346 76.927001) (xy 182.276655 108.077))
     (height -5.826961)
-    (gr_text "31.1500 mm" (at 189.252962 92.501708 270.0024095) (layer "F.SilkS")
+    (gr_text "31.1500 mm" (at 189.252962 92.501708 270.0024095) (layer "F.Fab")
       (effects (font (size 1 1) (thickness 0.15)))
     )
